File: Driverji.sch (KiCad schematic (older format))
At the start: 14 parts

Commit message: Dodal sheet z voltmetrom pod driverje
Parts:
- added C? (x2): CP, symbol Device:CP
- added C?: C1206, Passives:C1206M, symbol Passives:C1206
- added D?: LL4148, Diode_SMD:D_MiniMELF, symbol Diode:LL4148
Connections:
- net GND: now also U?.3 (COM), C?.2, C?.2
- net PWM_H: now reaches U?.1 (HIN)
- net PWM_L: now reaches U?.2 (LIN)
- net at U?.5 (VCC): now also C?.1, C?.1, D?.2 (A)
- net V_B: now reaches C?.1, U?.8 (VB)
- net V_B: now also C?.1, D?.1 (K)
- net Faza_Izhod renamed V_Izhod
- net V_Izhod: now also C?.2
Other:
- moved on the sheet: C?, U?
Changed lines of the file:
@@
 EESchema Schematic File Version 4
+LIBS:Seminar-cache
 EELAYER 26 0
 EELAYER END
 $Descr A4 11693 8268
 encoding utf-8
-Sheet 1 1
+Sheet 3 4
 Title ""
 Date ""
@@
 	6900 2850 6900 2450
 Text Label 10650 2450 0    50   ~ 0
-Faza_Izhod
+V_Izhod
 Wire Wire Line
 	10100 2450 10650 2450
@@
 L ICs:IR2181 U?
 U 1 1 5BC7B4E0
-P 1600 2400
-F 0 "U?" H 1600 2767 50  0000 C CNN
-F 1 "IR2181" H 1600 2676 50  0000 C CNN
-F 2 "Package_SO:SO8" H 1400 2650 50  0001 L CNN
-F 3 "http://www.irf.com/product-info/datasheets/data/ir2104.pdf" H 1400 2900 50  0001 L CNN
-	1    1600 2400
+P 2050 1900
+F 0 "U?" H 2050 2267 50  0000 C CNN
+F 1 "IR2181" H 2050 2176 50  0000 C CNN
+F 2 "Package_SO:SO8" H 1850 2150 50  0001 L CNN
+F 3 "http://www.irf.com/product-info/datasheets/data/ir2104.pdf" H 1850 2400 50  0001 L CNN
+	1    2050 1900
 	1    0    0    -1
 $EndComp
@@
 L Passives:C1206 C?
 U 1 1 5BC7CAD4
-P 2400 2400
-F 0 "C?" H 2515 2446 50  0000 L CNN
-F 1 "C1206" H 2515 2355 50  0000 L CNN
-F 2 "Passives:C1206M" H 2450 2300 50  0001 L CNN
-F 3 "" H 2400 2400 50  0001 C CNN
-	1    2400 2400
-	1    0    0    -1
-$EndComp
-Wire Wire Line
-	1900 2300 2400 2300
-Wire Wire Line
-	2400 2500 1900 2500
-Text Label 2100 2400 0    50   ~ 0
+P 2900 1700
+F 0 "C?" H 3015 1746 50  0000 L CNN
+F 1 "C1206" H 3015 1655 50  0000 L CNN
+F 2 "Passives:C1206M" H 2950 1600 50  0001 L CNN
+F 3 "" H 2900 1700 50  0001 C CNN
+	1    2900 1700
+	1    0    0    -1
+$EndComp
+Text Label 2550 1900 0    50   ~ 0
 Drv_H
-Text Label 2100 2600 0    50   ~ 0
+Text Label 2550 2100 0    50   ~ 0
 Drv_L
 Wire Wire Line
-	1900 2400 2100 2400
-Wire Wire Line
-	1900 2600 2100 2600
-Wire Wire Line
-	2950 2500 2400 2500
-Connection ~ 2400 2500
-Text Label 2950 2500 0    50   ~ 0
+	2350 1900 2550 1900
+Wire Wire Line
+	2350 2100 2550 2100
+Text Label 3400 2000 0    50   ~ 0
 V_S
 Text Label 5950 2450 2    50   ~ 0
@@
 Text Label 5950 3050 2    50   ~ 0
 Drv_L
+$Comp
+L Diode:LL4148 D?
+U 1 1 5BC720A0
+P 2100 1250
+F 0 "D?" H 2100 1034 50  0000 C CNN
+F 1 "LL4148" H 2100 1125 50  0000 C CNN
+F 2 "Diode_SMD:D_MiniMELF" H 2100 1075 50  0001 C CNN
+F 3 "http://www.vishay.com/docs/85557/ll4148.pdf" H 2100 1250 50  0001 C CNN
+	1    2100 1250
+	-1   0    0    1
+$EndComp
+Text Label 2550 1800 0    50   ~ 0
+V_B
+Wire Wire Line
+	2350 1800 2550 1800
+$Comp
+L Device:CP C?
+U 1 1 5BC7E67A
+P 3400 1700
+F 0 "C?" H 3518 1746 50  0000 L CNN
+F 1 "CP" H 3518 1655 50  0000 L CNN
+F 2 "" H 3438 1550 50  0001 C CNN
+F 3 "~" H 3400 1700 50  0001 C CNN
+	1    3400 1700
+	1    0    0    -1
+$EndComp
+Wire Wire Line
+	2900 1600 2900 1450
+Wire Wire Line
+	3400 1450 3400 1550
+Wire Wire Line
+	2900 1800 2900 2000
+Wire Wire Line
+	3400 2000 3400 1850
+Text Label 2900 1450 0    50   ~ 0
+V_B
+Wire Wire Line
+	2250 1250 2900 1250
+Text HLabel 900  1900 0    50   Input ~ 0
+PWM_H
+Text HLabel 900  2000 0    50   Input ~ 0
+PWM_L
+$Comp
+L Device:CP C?
+U 1 1 5BC8E650
+P 1450 1700
+F 0 "C?" H 1568 1746 50  0000 L CNN
+F 1 "CP" H 1568 1655 50  0000 L CNN
+F 2 "" H 1488 1550 50  0001 C CNN
+F 3 "~" H 1450 1700 50  0001 C CNN
+	1    1450 1700
+	1    0    0    -1
+$EndComp
+Wire Wire Line
+	1450 2100 1750 2100
+Wire Wire Line
+	1450 1850 1450 2100
+Wire Wire Line
+	1450 1150 1450 1250
+Connection ~ 1450 1450
+Wire Wire Line
+	1450 1450 1450 1550
+Wire Wire Line
+	1450 1450 1750 1450
+Wire Wire Line
+	1750 1450 1750 1800
+Wire Wire Line
+	1450 1250 1950 1250
+Connection ~ 1450 1250
+Wire Wire Line
+	1450 1250 1450 1450
+Wire Wire Line
+	2900 1250 2900 1450
+Connection ~ 2900 1450
+Wire Wire Line
+	2550 1800 2550 1450
+Wire Wire Line
+	2900 2000 3400 2000
+Wire Wire Line
+	2900 1450 3400 1450
+Wire Wire Line
+	2900 1450 2550 1450
+Wire Wire Line
+	2900 2000 2350 2000
+Connection ~ 2900 2000
+$Comp
+L Passives:C1206 C?
+U 1 1 5BCC0E27
+P 1000 1700
+F 0 "C?" H 1115 1746 50  0000 L CNN
+F 1 "C1206" H 1115 1655 50  0000 L CNN
+F 2 "Passives:C1206M" H 1050 1600 50  0001 L CNN
+F 3 "" H 1000 1700 50  0001 C CNN
+	1    1000 1700
+	1    0    0    -1
+$EndComp
+Wire Wire Line
+	1000 1600 1000 1450
+Wire Wire Line
+	900  1900 1750 1900
+Wire Wire Line
+	900  2000 1750 2000
+Wire Wire Line
+	1000 1800 1000 2100
+Wire Wire Line
+	1000 2100 1450 2100
+Connection ~ 1450 2100
+Wire Wire Line
+	1450 1450 1000 1450
+$Comp
+L Passives:GND #PWR?
+U 1 1 5BCC90C0
+P 1450 2300
+F 0 "#PWR?" H 1450 2150 50  0001 C CNN
+F 1 "GND" H 1600 2250 50  0001 C CNN
+F 2 "" H 1450 2300 50  0001 C CNN
+F 3 "" H 1450 2300 50  0001 C CNN
+	1    1450 2300
+	1    0    0    -1
+$EndComp
+Wire Wire Line
+	1450 2100 1450 2300
+$Sheet
+S 1450 3650 2100 1350
+U 5BCCBCD0
+F0 "V-meter1" 50
+F1 "V-Meter.sch" 50
+$EndSheet
+Text HLabel 1450 4050 2    50   Input ~ 0
+V_s
+Text HLabel 1450 4500 2    50   Input ~ 0
+GND
 $EndSCHEMATC

Commit message: Dokončal V-meter sheet in dodal A-meter sheet
Connections:
- net V_Izhod renamed Izhod1
Changed lines of the file:
@@
 $Descr A4 11693 8268
 encoding utf-8
-Sheet 3 4
+Sheet 3 5
 Title ""
 Date ""
@@
 	6900 2850 6900 2450
 Text Label 10650 2450 0    50   ~ 0
-V_Izhod
+Izhod1
 Wire Wire Line
 	10100 2450 10650 2450
@@
 Text HLabel 1450 4500 2    50   Input ~ 0
 GND
+$Sheet
+S 1450 5350 2100 1350
+U 5BCA57DE
+F0 "A-meter1" 50
+F1 "A_meter.sch" 50
+$EndSheet
+Text HLabel 3550 4300 0    50   Output ~ 0
+V_izm
+Text Label 10200 2450 0    50   ~ 0
+V_merjena
+Text HLabel 1450 5700 2    50   Input ~ 0
+Izhod
+Text HLabel 1450 6400 2    50   Input ~ 0
+GND
+Text HLabel 1450 6050 2    50   Input ~ 0
++5V
+Text HLabel 3550 5800 0    50   Input ~ 0
+Izhod_breme
+Text HLabel 3550 6200 0    50   Input ~ 0
+I_izm
 $EndSCHEMATC

Commit message: Dodano vezje za OC_trip pri merjenju toka
Connections:
- net Izhod1 renamed IzhodTranzistor
Other:
- moved on the sheet: Q?, R?

Commit message: Dodal nekaj blikornih kondenzatorjev
Parts:
- added C? (x2): C1206, Passives:C1206M, symbol Passives:C1206
- added C?: CP, symbol Device:CP
- added R? (x6): R1206, Passives:R1206M, symbol Passives:R1206
Connections:
- net +VDC: now also C?.1, C?.1, C?.1
- net GND: now also C?.2, C?.2, C?.2, R?.1, R?.1, R?.1
- net IzhodTranzistor: now also R?.1, R?.1, R?.1
- net at Q?.1 (G), R?.2: now also R?.2 (x5)
Other:
- moved on the sheet: Q?, R?
