File: Merjenje_DC_Napetosti.sch (KiCad schematic (older format))
At the start: 6 parts

Commit message: Dodal nekaj blikornih kondenzatorjev
Connections:
- wire segments 25 -> 23
Changed lines of the file:
@@
 Wire Wire Line
 	3500 2800 3500 2600
-Wire Wire Line
-	1800 1400 2800 1400
-Connection ~ 2800 1400
-Wire Wire Line
-	2800 2800 1800 2800
 Connection ~ 2800 2800
 Wire Wire Line
@@
 L Passives:GND #PWR?
 U 1 1 5BD4A769
-P 1800 2900
-F 0 "#PWR?" H 1800 2750 50  0001 C CNN
-F 1 "GND" H 1950 2850 50  0001 C CNN
-F 2 "" H 1800 2900 50  0001 C CNN
-F 3 "" H 1800 2900 50  0001 C CNN
-	1    1800 2900
+P 2800 2900
+F 0 "#PWR?" H 2800 2750 50  0001 C CNN
+F 1 "GND" H 2950 2850 50  0001 C CNN
+F 2 "" H 2800 2900 50  0001 C CNN
+F 3 "" H 2800 2900 50  0001 C CNN
+	1    2800 2900
 	1    0    0    -1
 $EndComp
 Wire Wire Line
-	1800 2900 1800 2800
+	2800 2900 2800 2800
 $Comp
 L power:+VDC #PWR?
 U 1 1 5BD8204F
-P 1800 1400
-F 0 "#PWR?" H 1800 1300 50  0001 C CNN
-F 1 "+VDC" H 1800 1675 50  0000 C CNN
-F 2 "" H 1800 1400 50  0001 C CNN
-F 3 "" H 1800 1400 50  0001 C CNN
-	1    1800 1400
+P 2800 1400
+F 0 "#PWR?" H 2800 1300 50  0001 C CNN
+F 1 "+VDC" H 2800 1675 50  0000 C CNN
+F 2 "" H 2800 1400 50  0001 C CNN
+F 3 "" H 2800 1400 50  0001 C CNN
+	1    2800 1400
 	1    0    0    -1
 $EndComp
+Connection ~ 2800 1400
 $EndSCHEMATC
