File: Merjenje_toka.sch (KiCad schematic (older format))
At the start: 7 parts

Commit message: Dodal nekaj blikornih kondenzatorjev
Parts:
- added C? (x5): C1206, Passives:C1206M, symbol Passives:C1206
Connections:
- net OC_trip is gone; now on net +3V3: U?.1, U?.1
- net +3V3: now also C?.1, C?.1
- net +5V: now also C?.1, C?.1
- net GND: now also C?.2, C?.2, C?.2, C?.2
Other:
- moved on the sheet: R?
Changed lines of the file:
@@
 L Passives:R1206 R?
 U 1 1 5BCACFE8
-P 6000 3700
-F 0 "R?" H 6000 3917 50  0000 C CNN
-F 1 "R1206" H 6000 3826 50  0000 C CNN
-F 2 "Passives:R1206M" H 5900 3600 50  0001 L CNN
-F 3 "" H 6000 3700 50  0001 C CNN
-	1    6000 3700
+P 6000 4150
+F 0 "R?" H 6000 4367 50  0000 C CNN
+F 1 "R1206" H 6000 4276 50  0000 C CNN
+F 2 "Passives:R1206M" H 5900 4050 50  0001 L CNN
+F 3 "" H 6000 4150 50  0001 C CNN
+	1    6000 4150
 	1    0    0    -1
 $EndComp
@@
 	4850 3300 5250 3300
 Wire Wire Line
-	5250 3300 5250 3700
-Wire Wire Line
-	5250 3700 5800 3700
+	5250 4150 5800 4150
 Connection ~ 5250 3300
 Wire Wire Line
 	5250 3300 5400 3300
-Wire Wire Line
-	6200 3700 6200 3200
-Wire Wire Line
-	6200 3200 6000 3200
 Text HLabel 7450 3200 2    50   Output ~ 0
 I_izm
@@
 L Passives:GND #PWR?
 U 1 1 5BCAD7C1
-P 5600 3550
-F 0 "#PWR?" H 5600 3400 50  0001 C CNN
-F 1 "GND" H 5750 3500 50  0001 C CNN
-F 2 "" H 5600 3550 50  0001 C CNN
-F 3 "" H 5600 3550 50  0001 C CNN
-	1    5600 3550
-	1    0    0    -1
-$EndComp
-Wire Wire Line
-	5600 3550 5600 3500
+P 5600 3750
+F 0 "#PWR?" H 5600 3600 50  0001 C CNN
+F 1 "GND" H 5750 3700 50  0001 C CNN
+F 2 "" H 5600 3750 50  0001 C CNN
+F 3 "" H 5600 3750 50  0001 C CNN
+	1    5600 3750
+	1    0    0    -1
+$EndComp
 $Comp
 L power:+5V #PWR?
@@
 $EndComp
 Wire Wire Line
-	5600 2750 5600 2900
+	5600 2750 5600 2800
 $Comp
 L Passives:R1206 R?
@@
 L Passives:GND #PWR?
 U 1 1 5BCDDCB8
-P 7150 1650
-F 0 "#PWR?" H 7150 1500 50  0001 C CNN
-F 1 "GND" H 7300 1600 50  0001 C CNN
-F 2 "" H 7150 1650 50  0001 C CNN
-F 3 "" H 7150 1650 50  0001 C CNN
-	1    7150 1650
-	1    0    0    -1
-$EndComp
-Wire Wire Line
-	7150 1650 7150 1600
+P 7150 1700
+F 0 "#PWR?" H 7150 1550 50  0001 C CNN
+F 1 "GND" H 7300 1650 50  0001 C CNN
+F 2 "" H 7150 1700 50  0001 C CNN
+F 3 "" H 7150 1700 50  0001 C CNN
+	1    7150 1700
+	1    0    0    -1
+$EndComp
 $Comp
 L Passives:GND #PWR?
@@
 $EndComp
 Wire Wire Line
-	7150 2800 7150 2700
+	7150 2800 7150 2750
 Text HLabel 6500 1200 0    50   Input ~ 0
 U_max
@@
 $EndComp
 Wire Wire Line
-	7150 900  7150 1000
-Wire Wire Line
-	7150 2000 7150 2100
+	7150 900  7150 950
+Wire Wire Line
+	7150 2000 7150 2050
 Wire Wire Line
 	5100 3100 5100 3800
@@
 	1    0    0    -1
 $EndComp
+$Comp
+L Passives:C1206 C?
+U 1 1 5BE2D76B
+P 6050 3550
+F 0 "C?" H 6165 3596 50  0000 L CNN
+F 1 "C1206" H 6165 3505 50  0000 L CNN
+F 2 "Passives:C1206M" H 6100 3450 50  0001 L CNN
+F 3 "" H 6050 3550 50  0001 C CNN
+	1    6050 3550
+	1    0    0    -1
+$EndComp
+Wire Wire Line
+	6200 3200 6000 3200
+Wire Wire Line
+	6200 3200 6200 4150
+Wire Wire Line
+	5250 3300 5250 4150
+Wire Wire Line
+	5600 3500 5600 3700
+Wire Wire Line
+	5600 3700 6050 3700
+Wire Wire Line
+	6050 3700 6050 3650
+Connection ~ 5600 3700
+Wire Wire Line
+	5600 3700 5600 3750
+Wire Wire Line
+	6050 2800 5600 2800
+Wire Wire Line
+	6050 2800 6050 3450
+Connection ~ 5600 2800
+Wire Wire Line
+	5600 2800 5600 2900
+$Comp
+L Passives:C1206 C?
+U 1 1 5BE345EB
+P 8550 2650
+F 0 "C?" H 8665 2696 50  0000 L CNN
+F 1 "C1206" H 8665 2605 50  0000 L CNN
+F 2 "Passives:C1206M" H 8600 2550 50  0001 L CNN
+F 3 "" H 8550 2650 50  0001 C CNN
+	1    8550 2650
+	1    0    0    -1
+$EndComp
+$Comp
+L Passives:C1206 C?
+U 1 1 5BE36614
+P 7550 2600
+F 0 "C?" H 7665 2646 50  0000 L CNN
+F 1 "C1206" H 7665 2555 50  0000 L CNN
+F 2 "Passives:C1206M" H 7600 2500 50  0001 L CNN
+F 3 "" H 7550 2600 50  0001 C CNN
+	1    7550 2600
+	1    0    0    -1
+$EndComp
+Wire Wire Line
+	7150 2750 7550 2750
+Wire Wire Line
+	7550 2750 7550 2700
+Connection ~ 7150 2750
+Wire Wire Line
+	7150 2750 7150 2700
+Wire Wire Line
+	7550 2500 7550 2400
+Wire Wire Line
+	7550 2050 7150 2050
+Connection ~ 7550 2400
+Wire Wire Line
+	7550 2400 7550 2050
+Connection ~ 7150 2050
+Wire Wire Line
+	7150 2050 7150 2100
+$Comp
+L Passives:C1206 C?
+U 1 1 5BE3C85C
+P 7600 1550
+F 0 "C?" H 7715 1596 50  0000 L CNN
+F 1 "C1206" H 7715 1505 50  0000 L CNN
+F 2 "Passives:C1206M" H 7650 1450 50  0001 L CNN
+F 3 "" H 7600 1550 50  0001 C CNN
+	1    7600 1550
+	1    0    0    -1
+$EndComp
+Wire Wire Line
+	7150 1600 7150 1650
+Wire Wire Line
+	7150 1650 7600 1650
+Connection ~ 7150 1650
+Wire Wire Line
+	7150 1650 7150 1700
+Wire Wire Line
+	7600 1450 7600 950
+Wire Wire Line
+	7600 950  7150 950
+Connection ~ 7150 950
+Wire Wire Line
+	7150 950  7150 1000
+$Comp
+L Passives:C1206 C?
+U 1 1 5BE3FC8E
+P 2000 3300
+F 0 "C?" H 2115 3346 50  0000 L CNN
+F 1 "C1206" H 2115 3255 50  0000 L CNN
+F 2 "Passives:C1206M" H 2050 3200 50  0001 L CNN
+F 3 "" H 2000 3300 50  0001 C CNN
+	1    2000 3300
+	1    0    0    -1
+$EndComp
+Wire Wire Line
+	2000 3400 2200 3400
+Connection ~ 2200 3400
+Wire Wire Line
+	2200 3200 2000 3200
+Connection ~ 2200 3200
 $EndSCHEMATC
